Commit message: new file

File: description/robot_core.xacro (robot description, xacro)
@@ -14,3 +14,17 @@
     </material>
     <link name="base_link"></link>
+    <joint name="chassis_joint" type="fixed">
+        <parent link="base_link"/>
+        <child link="chassis_link"/>
+        <origin xyz="-0.1 0.0 0.0"/>
+    </joint>
+    <link name="chassis_link">
+        <visual>
+            <origin xyz="0.15 0.0 0.075"/>
+            <geometry>
+                <box size="0.3 0.3 0.15"/>
+            </geometry>
+            <material name="white"/>
+        </visual>
+    </link>
 </robot>

Commit message: change:

File: description/robot_core.xacro (robot description, xacro)
@@ -41,4 +41,7 @@
         </xacro:inertial_box>
     </link>
+    <gazebo reference="chassis_link">
+        <material>Gazebo/White</material>
+    </gazebo>
     <!-- LEFT FORWARD WHEEL -->
     <joint name="left_forward_wheel_joint" type="continuous">
@@ -64,4 +67,7 @@
         </xacro:inertial_cylinder>
     </link>
+    <gazebo reference="left_forward_wheel_link">
+        <material>Gazebo/Blue</material>
+    </gazebo>
     <!-- RIGHT FORWARD WHEEL -->
     <joint name="right_forward_wheel_joint" type="continuous">
@@ -87,4 +93,7 @@
         </xacro:inertial_cylinder>
     </link>
+    <gazebo reference="right_forward_wheel_link">
+        <material>Gazebo/Red</material>
+    </gazebo>
     <!-- LEFT REAR WHEEL -->
     <joint name="left_rear_wheel_joint" type="continuous">
@@ -110,4 +119,7 @@
         </xacro:inertial_cylinder>
     </link>
+    <gazebo reference="left_rear_wheel_link">
+        <material>Gazebo/Red</material>
+    </gazebo>
     <!-- RIGHT REAR WHEEL -->
     <joint name="right_rear_wheel_joint" type="continuous">
@@ -133,3 +145,6 @@
         </xacro:inertial_cylinder>
     </link>
+    <gazebo reference="right_rear_wheel_link">
+        <material>Gazebo/Blue</material>
+    </gazebo>
 </robot>
