Commit message: change: link name

File: description/lidar.xacro (robot description, xacro)
@@ -3,8 +3,8 @@
     <joint name="laser_joint" type="fixed">
         <parent link="chassis_link"/>
-        <child link="laser_link"/>
-        <origin xyz="0.1  0.0 0.175" rpy="0.0 0.0 0.0"/>
+        <child link="laser_frame"/>
+        <origin xyz="0.04 0.0 0.04" rpy="0.0 0.0 0.0"/>
     </joint>
-    <link name="laser_link">
+    <link name="laser_frame">
         <visual>
             <geometry>
@@ -22,9 +22,9 @@
         </xacro:inertial_cylinder>
     </link>
-    <gazebo reference="laser_link">
+    <gazebo reference="laser_frame">
         <material>Gazebo/Orange</material>
         <sensor name="laser" type="ray">
             <pose> 0 0 0 0 0 0 </pose>
-            <visualize>false</visualize>
+            <visualize>true</visualize>
             <update_rate>10</update_rate>
             <ray>

Commit message: add: camera

File: description/lidar.xacro (robot description, xacro)
@@ -4,5 +4,5 @@
         <parent link="chassis_link"/>
         <child link="laser_frame"/>
-        <origin xyz="0.04 0.0 0.04" rpy="0.0 0.0 0.0"/>
+        <origin xyz="-0.1 0.0 0.04" rpy="0.0 0.0 0.0"/>
     </joint>
     <link name="laser_frame">

Commit message: add: camera

File: description/lidar.xacro (robot description, xacro)
@@ -4,5 +4,5 @@
         <parent link="chassis_link"/>
         <child link="laser_frame"/>
-        <origin xyz="-0.1 0.0 0.04" rpy="0.0 0.0 0.0"/>
+        <origin xyz="0.1 0.0 0.07" rpy="0.0 0.0 0.0"/>
     </joint>
     <link name="laser_frame">

File: description/robot.urdf.xacro (robot description, xacro)
@@ -4,3 +4,4 @@
     <xacro:include filename="gazebo_control.xacro"/>
     <xacro:include filename="lidar.xacro"/>
+    <xacro:include filename="camera.xacro"/>
 </robot>
