Commit message: change: change to real size

File: description/camera.xacro (robot description, xacro)
@@ -4,5 +4,5 @@
         <parent link="chassis_link"/>
         <child link="camera_link"/>
-        <origin xyz="-0.01 0.0 0.04" rpy="0.0 0.0 0.0"/>
+        <origin xyz="0.01 0.0 0.04" rpy="0.0 0.0 0.0"/>
     </joint>
     <link name="camera_link">

File: description/lidar.xacro (robot description, xacro)
@@ -4,10 +4,10 @@
         <parent link="chassis_link"/>
         <child link="laser_frame"/>
-        <origin xyz="0.1 0.0 0.07" rpy="0.0 0.0 0.0"/>
+        <origin xyz="0.0 0.0 0.07" rpy="0.0 0.0 0.0"/>
     </joint>
     <link name="laser_frame">
         <visual>
             <geometry>
-                <cylinder radius="0.05" length="0.04"/>
+                <cylinder radius="0.035" length="0.06"/>
             </geometry>
             <material name="orange"/>
@@ -15,5 +15,5 @@
         <collision>
             <geometry>
-                <cylinder radius="0.0" length="0.0"/>
+                <cylinder radius="0.035" length="0.06"/>
             </geometry>
         </collision>

File: description/robot_core.xacro (robot description, xacro)
@@ -21,22 +21,22 @@
         <parent link="base_link"/>
         <child link="chassis_link"/>
-        <origin xyz="-0.1 0.0 0.0"/>
+        <origin xyz="0.3 0.0 0.0"/>
     </joint>
     <link name="chassis_link">
         <visual>
-            <origin xyz="0.15 0.0 0.005"/>
+            <origin xyz="0.0 0.0 0.0"/>
             <geometry>
-                <box size="0.3 0.3 0.01"/>
+                <box size="0.26 0.16 0.01"/>
             </geometry>
             <material name="white"/>
         </visual>
         <collision>
-            <origin xyz="0.15 0.0 0.005"/>
+            <origin xyz="0.0 0.0 0.0"/>
             <geometry>
-                <box size="0.3 0.3 0.01"/>
+                <box size="0.26 0.16 0.01"/>
             </geometry>
         </collision>
-        <xacro:inertial_box mass="0.5" x="0.3" y="0.3" z="0.01">
-            <origin xyz="0.15 00. 0.075" rpy="0.0 0.0 0.0"/>
+        <xacro:inertial_box mass="0.5" x="0.26" y="0.16" z="0.01">
+            <origin xyz="0.0 0.0 0.0" rpy="0.0 0.0 0.0"/>
         </xacro:inertial_box>
     </link>
@@ -48,5 +48,5 @@
         <parent link="chassis_link"/>
         <child link="left_forward_wheel_link"/>
-        <origin xyz="0.03 0.175 0.0" rpy="-${pi/2} 0.0 0.0"/>
+        <origin xyz="0.115 0.07 0.0" rpy="-${pi/2} 0.0 0.0"/>
         <axis xyz="0.0 0.0 1"/>
     </joint>
@@ -74,5 +74,5 @@
         <parent link="chassis_link"/>
         <child link="right_forward_wheel_link"/>
-        <origin xyz="0.03 -0.175 0.0" rpy="${pi/2} 0.0 0.0"/>
+        <origin xyz="0.115 -0.07 0.0" rpy="${pi/2} 0.0 0.0"/>
         <axis xyz="0.0 0.0 -1"/>
     </joint>
@@ -100,5 +100,5 @@
         <parent link="chassis_link"/>
         <child link="left_rear_wheel_link"/>
-        <origin xyz="0.27 0.175 0.0" rpy="-${pi/2} 0.0 0.0"/>
+        <origin xyz="-0.115 0.07 0.0" rpy="-${pi/2} 0.0 0.0"/>
         <axis xyz="0.0 0.0 1"/>
     </joint>
@@ -126,5 +126,5 @@
         <parent link="chassis_link"/>
         <child link="right_rear_wheel_link"/>
-        <origin xyz="0.27 -0.175 0.0" rpy="${pi/2} 0.0 0.0"/>
+        <origin xyz="-0.115 -0.07 0.0" rpy="${pi/2} 0.0 0.0"/>
         <axis xyz="0.0 0.0 -1"/>
     </joint>

Commit message: change: values changed to real

File: description/camera.xacro (robot description, xacro)
@@ -4,5 +4,5 @@
         <parent link="chassis_link"/>
         <child link="camera_link"/>
-        <origin xyz="0.01 0.0 0.04" rpy="0.0 0.0 0.0"/>
+        <origin xyz="0.14 0.0 0.04" rpy="0.0 0.0 0.0"/>
     </joint>
     <link name="camera_link">

File: description/robot_core.xacro (robot description, xacro)
@@ -17,4 +17,13 @@
         <color rgba="0 0 0 1"/>
     </material>
+    <xacro:property name="chassis_length" value="0.26"/>
+    <xacro:property name="chassis_width" value="0.16"/>
+    <xacro:property name="chassis_height" value="0.01"/>
+    <xacro:property name="wheel_radius" value="0.03"/>
+    <xacro:property name="wheel_length" value="0.03"/>
+    <xacro:property name="wheel_offset_x" value="0.115"/>
+    <xacro:property name="wheel_offset_y" value="0.105"/>
+    <xacro:property name="wheel_offset_z" value="0.02"/>
+    <xacro:property name="wheel_mass" value="0.01"/>
     <link name="base_link"></link>
     <joint name="chassis_joint" type="fixed">
@@ -27,5 +36,5 @@
             <origin xyz="0.0 0.0 0.0"/>
             <geometry>
-                <box size="0.26 0.16 0.01"/>
+                <box size="${chassis_length} ${chassis_width} ${chassis_height}"/>
             </geometry>
             <material name="white"/>
@@ -34,8 +43,8 @@
             <origin xyz="0.0 0.0 0.0"/>
             <geometry>
-                <box size="0.26 0.16 0.01"/>
+                <box size="${chassis_length} ${chassis_width} ${chassis_height}"/>
             </geometry>
         </collision>
-        <xacro:inertial_box mass="0.5" x="0.26" y="0.16" z="0.01">
+        <xacro:inertial_box mass="0.5" x="${chassis_length}" y="${chassis_width}" z="${chassis_height}">
             <origin xyz="0.0 0.0 0.0" rpy="0.0 0.0 0.0"/>
         </xacro:inertial_box>
@@ -48,5 +57,5 @@
         <parent link="chassis_link"/>
         <child link="left_forward_wheel_link"/>
-        <origin xyz="0.115 0.07 0.0" rpy="-${pi/2} 0.0 0.0"/>
+        <origin xyz="${wheel_offset_x} ${wheel_offset_y} ${-wheel_offset_z}" rpy="-${pi/2} 0.0 0.0"/>
         <axis xyz="0.0 0.0 1"/>
     </joint>
@@ -54,5 +63,5 @@
         <visual>
             <geometry>
-                <cylinder radius="0.03" length="0.03"/>
+                <cylinder radius="${wheel_radius}" length="${wheel_length}"/>
             </geometry>
             <material name="blue"/>
@@ -60,8 +69,8 @@
         <collision>
             <geometry>
-                <cylinder radius="0.03" length="0.03"/>
+                <cylinder radius="${wheel_radius}" length="${wheel_length}"/>
             </geometry>
         </collision>
-        <xacro:inertial_cylinder mass="0.1" length="0.06" radius="0.03">
+        <xacro:inertial_cylinder mass="${wheel_mass}" length="${wheel_length}" radius="${wheel_radius}">
             <origin xyz="0.0 0.0 0.0" rpy="0.0 0.0 0.0"/>
         </xacro:inertial_cylinder>
@@ -74,5 +83,5 @@
         <parent link="chassis_link"/>
         <child link="right_forward_wheel_link"/>
-        <origin xyz="0.115 -0.07 0.0" rpy="${pi/2} 0.0 0.0"/>
+        <origin xyz="${wheel_offset_x} ${-wheel_offset_y} ${-wheel_offset_z}" rpy="${pi/2} 0.0 0.0"/>
         <axis xyz="0.0 0.0 -1"/>
     </joint>
@@ -80,5 +89,5 @@
         <visual>
             <geometry>
-                <cylinder radius="0.03" length="0.03"/>
+                <cylinder radius="${wheel_radius}" length="${wheel_length}"/>
             </geometry>
             <material name="red"/>
@@ -86,8 +95,8 @@
         <collision>
             <geometry>
-                <cylinder radius="0.03" length="0.03"/>
+                <cylinder radius="${wheel_radius}" length="${wheel_length}"/>
             </geometry>
         </collision>
-        <xacro:inertial_cylinder mass="0.1" length="0.06" radius="0.03">
+        <xacro:inertial_cylinder mass="${wheel_mass}" length="${wheel_length}" radius="${wheel_radius}">
             <origin xyz="0.0 0.0 0.0" rpy="0.0 0.0 0.0"/>
         </xacro:inertial_cylinder>
@@ -100,5 +109,5 @@
         <parent link="chassis_link"/>
         <child link="left_rear_wheel_link"/>
-        <origin xyz="-0.115 0.07 0.0" rpy="-${pi/2} 0.0 0.0"/>
+        <origin xyz="${-wheel_offset_x} ${wheel_offset_y} ${-wheel_offset_z}" rpy="-${pi/2} 0.0 0.0"/>
         <axis xyz="0.0 0.0 1"/>
     </joint>
@@ -106,5 +115,5 @@
         <visual>
             <geometry>
-                <cylinder radius="0.03" length="0.03"/>
+                <cylinder radius="${wheel_radius}" length="${wheel_length}"/>
             </geometry>
             <material name="red"/>
@@ -112,8 +121,8 @@
         <collision>
             <geometry>
-                <cylinder radius="0.03" length="0.03"/>
+                <cylinder radius="${wheel_radius}" length="${wheel_length}"/>
             </geometry>
         </collision>
-        <xacro:inertial_cylinder mass="0.1" length="0.06" radius="0.03">
+        <xacro:inertial_cylinder mass="${wheel_mass}" length="${wheel_length}" radius="${wheel_radius}">
             <origin xyz="0.0 0.0 0.0" rpy="0.0 0.0 0.0"/>
         </xacro:inertial_cylinder>
@@ -126,5 +135,5 @@
         <parent link="chassis_link"/>
         <child link="right_rear_wheel_link"/>
-        <origin xyz="-0.115 -0.07 0.0" rpy="${pi/2} 0.0 0.0"/>
+        <origin xyz="${-wheel_offset_x} ${-wheel_offset_y} ${-wheel_offset_z}" rpy="${pi/2} 0.0 0.0"/>
         <axis xyz="0.0 0.0 -1"/>
     </joint>
@@ -132,5 +141,5 @@
         <visual>
             <geometry>
-                <cylinder radius="0.03" length="0.03"/>
+                <cylinder radius="${wheel_radius}" length="${wheel_length}"/>
             </geometry>
             <material name="blue"/>
@@ -138,8 +147,8 @@
         <collision>
             <geometry>
-                <cylinder radius="0.03" length="0.03"/>
+                <cylinder radius="${wheel_radius}" length="${wheel_length}"/>
             </geometry>
         </collision>
-        <xacro:inertial_cylinder mass="0.1" length="0.06" radius="0.03">
+        <xacro:inertial_cylinder mass="${wheel_mass}" length="${wheel_length}" radius="${wheel_radius}">
             <origin xyz="0.0 0.0 0.0" rpy="0.0 0.0 0.0"/>
         </xacro:inertial_cylinder>
