Commit message: add: xacro

File: description/robot.urdf.xacro (robot description, xacro)
@@ -1,5 +1,4 @@
 <?xml version="1.0"?>
 <<robot xmlns:xacro="http://www.ros.org/wiki/xacro" name="robot">
-    <link name="base_link">
-    </link>
+    <xacro:include filename="robot_core.xacro"/>
 </robot>

Commit message: new file: inertial_macros

File: description/robot.urdf.xacro (robot description, xacro)
@@ -1,4 +1,4 @@
 <?xml version="1.0"?>
-<<robot xmlns:xacro="http://www.ros.org/wiki/xacro" name="robot">
+<robot xmlns:xacro="http://www.ros.org/wiki/xacro" name="robot">
     <xacro:include filename="robot_core.xacro"/>
 </robot>

File: description/robot_core.xacro (robot description, xacro)
@@ -1,4 +1,5 @@
 <?xml version="1.0"?>
 <robot xmlns:xacro="http://www.ros.org/wiki/xacro">
+    <xacro:include filename="inertial_macros.xacro"/>
     <material name="white">
         <color rgba="1 1 1 1"/>
@@ -9,4 +10,7 @@
     <material name="blue">
         <color rgba="0.2 0.2 1 1"/>
+    </material>
+    <material name="red">
+        <color rgba="1 0.2 0.2 1"/>
     </material>
     <material name="black">
@@ -21,10 +25,111 @@
     <link name="chassis_link">
         <visual>
-            <origin xyz="0.15 0.0 0.075"/>
+            <origin xyz="0.15 0.0 0.005"/>
             <geometry>
-                <box size="0.3 0.3 0.15"/>
+                <box size="0.3 0.3 0.01"/>
             </geometry>
             <material name="white"/>
         </visual>
+        <collision>
+            <origin xyz="0.15 0.0 0.005"/>
+            <geometry>
+                <box size="0.3 0.3 0.01"/>
+            </geometry>
+        </collision>
+        <xacro:inertial_box mass="0.5" x="0.3" y="0.3" z="0.01">
+            <origin xyz="0.15 00. 0.075" rpy="0.0 0.0 0.0"/>
+        <xacro:inertial_box>
+    </link>
+    <!-- LEFT FORWARD WHEEL -->
+    <joint name="left_forward_wheel_joint" type="continuous">
+        <parent link="chassis_link"/>
+        <child link="left_forward_wheel_link"/>
+        <origin xyz="0.03 0.175 0.0" rpy="-${pi/2} 0.0 0.0"/>
+        <axis xyz="0.0 0.0 1"/>
+    </joint>
+    <link name="left_forward_wheel_link">
+        <visual>
+            <geometry>
+                <cylinder radius="0.03" length="0.03"/>
+            </geometry>
+            <material name="blue"/>
+        </visual>
+        <collision>
+            <geometry>
+                <cylinder radius="0.03" length="0.03"/>
+            </geometry>
+        </collision>
+        <xacro:inertial_box mass="0.1" length="0.06" radius="0.03">
+            <origin xyz="0.0 0.0 0.0" rpy="0.0 0.0 0.0"/>
+        <xacro:inertial_box>
+    </link>
+    <!-- RIGHT FORWARD WHEEL -->
+    <joint name="right_forward_wheel_joint" type="continuous">
+        <parent link="chassis_link"/>
+        <child link="right_forward_wheel_link"/>
+        <origin xyz="0.03 -0.175 0.0" rpy="${pi/2} 0.0 0.0"/>
+        <axis xyz="0.0 0.0 -1"/>
+    </joint>
+    <link name="right_forward_wheel_link">
+        <visual>
+            <geometry>
+                <cylinder radius="0.03" length="0.03"/>
+            </geometry>
+            <material name="red"/>
+        </visual>
+        <collision>
+            <geometry>
+                <cylinder radius="0.03" length="0.03"/>
+            </geometry>
+        </collision>
+        <xacro:inertial_box mass="0.1" length="0.06" radius="0.03">
+            <origin xyz="0.0 0.0 0.0" rpy="0.0 0.0 0.0"/>
+        <xacro:inertial_box>
+    </link>
+    <!-- LEFT REAR WHEEL -->
+    <joint name="left_rear_wheel_joint" type="continuous">
+        <parent link="chassis_link"/>
+        <child link="left_rear_wheel_link"/>
+        <origin xyz="0.27 0.175 0.0" rpy="-${pi/2} 0.0 0.0"/>
+        <axis xyz="0.0 0.0 1"/>
+    </joint>
+    <link name="left_rear_wheel_link">
+        <visual>
+            <geometry>
+                <cylinder radius="0.03" length="0.03"/>
+            </geometry>
+            <material name="red"/>
+        </visual>
+        <collision>
+            <geometry>
+                <cylinder radius="0.03" length="0.03"/>
+            </geometry>
+        </collision>
+        <xacro:inertial_box mass="0.1" length="0.06" radius="0.03">
+            <origin xyz="0.0 0.0 0.0" rpy="0.0 0.0 0.0"/>
+        <xacro:inertial_box>
+    </link>
+    <!-- RIGHT REAR WHEEL -->
+    <joint name="right_rear_wheel_joint" type="continuous">
+        <parent link="chassis_link"/>
+        <child link="right_rear_wheel_link"/>
+        <origin xyz="0.27 -0.175 0.0" rpy="${pi/2} 0.0 0.0"/>
+        <axis xyz="0.0 0.0 -1"/>
+    </joint>
+    <link name="right_rear_wheel_link">
+        <visual>
+            <geometry>
+                <cylinder radius="0.03" length="0.03"/>
+            </geometry>
+            <material name="blue"/>
+        </visual>
+        <collision>
+            <geometry>
+                <cylinder radius="0.03" length="0.03"/>
+            </geometry>
+        </collision>
+        <xacro:inertial_box mass="0.1" length="0.06" radius="0.03">
+            <origin xyz="0.0 0.0 0.0" rpy="0.0 0.0 0.0"/>
+        <xacro:inertial_box>
     </link>
 </robot>

Commit message: change:

File: description/robot.urdf.xacro (robot description, xacro)
@@ -1,8 +1,13 @@
 <?xml version="1.0"?>
 <robot xmlns:xacro="http://www.ros.org/wiki/xacro" name="robot">
+    <xacro:arg name="use_ros2_control" default="true"/>
     <xacro:include filename="robot_core.xacro"/>
-    <!-- <xacro:include filename="gazebo_control.xacro"/> -->
+    <xacro:if value="$(arg use_ros2_control)">
+        <xacro:include filename="ros2_control.xacro"/>
+    </xacro:if>
+    <xacro:unless value="$(arg use_ros2_control)">
+        <xacro:include filename="gazebo_control.xacro"/>
+    </xacro:unless>
     <xacro:include filename="lidar.xacro"/>
     <xacro:include filename="camera.xacro"/>
-    <xacro:include filename="ros2_control.xacro"/>
 </robot>

File: description/robot_core.xacro (robot description, xacro)
@@ -69,5 +69,5 @@
         <collision>
             <geometry>
-                <cylinder radius="${wheel_radius}" length="${wheel_length}"/>
+                <sphere radius="${wheel_radius}" length="${wheel_length}"/>
             </geometry>
         </collision>
@@ -95,5 +95,5 @@
         <collision>
             <geometry>
-                <cylinder radius="${wheel_radius}" length="${wheel_length}"/>
+                <sphere radius="${wheel_radius}" length="${wheel_length}"/>
             </geometry>
         </collision>
@@ -121,5 +121,5 @@
         <collision>
             <geometry>
-                <cylinder radius="${wheel_radius}" length="${wheel_length}"/>
+                <sphere radius="${wheel_radius}" length="${wheel_length}"/>
             </geometry>
         </collision>
@@ -147,5 +147,5 @@
         <collision>
             <geometry>
-                <cylinder radius="${wheel_radius}" length="${wheel_length}"/>
+                <sphere radius="${wheel_radius}" length="${wheel_length}"/>
             </geometry>
         </collision>
